Commit message: update

File: RobotSim/assets/so100/urdf/so_arm100.urdf (robot description, URDF)
Before this commit: robot so_100_arm, 8 links, 7 joints
Links:
- link Base: geometry collision mesh filename=/public/xingyuezhao/zhy/RobotSim/assets/Base.STL; visual mesh filename=/public/xingyuezhao/zhy/RobotSim/assets/Base.STL
- link Fixed_Gripper: geometry collision mesh filename=/public/xingyuezhao/zhy/RobotSim/assets/Fixed_Gripper.STL; visual mesh filename=/public/xingyuezhao/zhy/RobotSim/assets/Fixed_Gripper.STL
- link Lower_Arm: geometry collision mesh filename=/public/xingyuezhao/zhy/RobotSim/assets/Lower_Arm.STL; visual mesh filename=/public/xingyuezhao/zhy/RobotSim/assets/Lower_Arm.STL
- link Moving_Jaw: geometry collision mesh filename=/public/xingyuezhao/zhy/RobotSim/assets/Moving_Jaw.STL; visual mesh filename=/public/xingyuezhao/zhy/RobotSim/assets/Moving_Jaw.STL
- link Shoulder_Rotation_Pitch: geometry collision mesh filename=/public/xingyuezhao/zhy/RobotSim/assets/Shoulder_Rotation_P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; visual mesh filename=/public/xingyuezhao/zhy/RobotSim/assets/Shoulder_Rotation_P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
- link Upper_Arm: geometry collision mesh filename=/public/xingyuezhao/zhy/RobotSim/assets/Upper_Arm.STL; visual mesh filename=/public/xingyuezhao/zhy/RobotSim/assets/Upper_Arm.STL
- link Wrist_Pitch_Roll: geometry collision mesh filename=/public/xingyuezhao/zhy/RobotSim/assets/Wrist_Pitch_Roll.STL; visual mesh filename=/public/xingyuezhao/zhy/RobotSim/assets/Wrist_Pitch_Roll.STL
